File: KiCAD/STM32 RC AUTO MOZEK/STM32 RC AUTO MOZEK.kicad_pcb (KiCad board)
At the start: 2 copper layers, 30 parts, among them J1 Conn_01x02_Socket, J2 Conn_01x02_Socket, J3 Conn_01x02_Socket, J4 Conn_01x02_Socket, J5 Conn_01x02_Socket, J6 Conn_01x02_Socket, J7 Conn_01x02_Socket, J8 Conn_01x03_Socket, J9 Conn_01x03_Socket, U1 LD1117S33TR_SOT223, U10 ACS712xLCTR-20A, U11 ACS712xLCTR-20A, U12 STM32F411RCTx, U13 STM32F030C8Tx, U2 SHT4x, U2 STM32C031C6Ux, U3 L7805, U4 ACS712xLCTR-20A, U4 L7808, U5 NRF24L01_Breakout, U6 NRF24L01_Breakout, U7 ACS712xLCTR-20A, U8 ACS712xLCTR-20A, U9 ACS712xLCTR-20A

Commit message: .
Parts:
- removed J7: Conn_01x02_Socket, Connector_Wire:SolderWire-2sqmm_1x02_P7.8mm_D2mm_OD3.9mm_Relief
- removed U2: STM32C031C6Ux, Package_DFN_QFN:QFN-48-1EP_7x7mm_P0.5mm_EP5.6x5.6mm
- removed U2: SHT4x, Sensor_Humidity:Sensirion_DFN-4_1.5x1.5mm_P0.8mm_SHT4x_NoCentralPad
- removed the U4 at (113.0, 58.6)
- removed the U4 at (64.2, 53.2)
- added C1: C, Capacitor_SMD:C_0805_2012Metric_Pad1.18x1.45mm_HandSolder, F.Cu at (53.6, 69.9)
- added C10: 12,5pF, Capacitor_SMD:C_0805_2012Metric_Pad1.18x1.45mm_HandSolder, F.Cu at (58.5, 81.9)
- added C11: 12,5pF, Capacitor_SMD:C_0805_2012Metric_Pad1.18x1.45mm_HandSolder, F.Cu at (35.7, 105.2)
- added C12: 12,5pF, Capacitor_SMD:C_0805_2012Metric_Pad1.18x1.45mm_HandSolder, F.Cu at (38.7, 105.2)
- added C13: 12,5pF, Capacitor_SMD:C_0805_2012Metric_Pad1.18x1.45mm_HandSolder, F.Cu at (41.7, 105.2)
- added C14: 12,5pF, Capacitor_SMD:C_0805_2012Metric_Pad1.18x1.45mm_HandSolder, F.Cu at (44.7, 105.2)
- added C2: C, Capacitor_SMD:C_0805_2012Metric_Pad1.18x1.45mm_HandSolder, F.Cu at (53.6, 72.9)
- added C3: C, Capacitor_SMD:C_0805_2012Metric_Pad1.18x1.45mm_HandSolder, F.Cu at (53.6, 75.9)
- added C4: C, Capacitor_SMD:C_0805_2012Metric_Pad1.18x1.45mm_HandSolder, F.Cu at (53.6, 78.9)
- added C5: C, Capacitor_SMD:C_0805_2012Metric_Pad1.18x1.45mm_HandSolder, F.Cu at (53.6, 81.9)
- added C6: C, Capacitor_SMD:C_0805_2012Metric_Pad1.18x1.45mm_HandSolder, F.Cu at (58.5, 69.9)
- added C7: 12,5pF, Capacitor_SMD:C_0805_2012Metric_Pad1.18x1.45mm_HandSolder, F.Cu at (58.5, 72.9)
- added C8: 12,5pF, Capacitor_SMD:C_0805_2012Metric_Pad1.18x1.45mm_HandSolder, F.Cu at (58.5, 75.9)
- added C9: 12,5pF, Capacitor_SMD:C_0805_2012Metric_Pad1.18x1.45mm_HandSolder, F.Cu at (58.5, 78.9)
- added J10: Conn_01x05_Socket, Connector_Wire:SolderWire-0.5sqmm_1x05_P4.8mm_D0.9mm_OD2.3mm_Relief, F.Cu at (152.4, 133.5)
- added J11: Conn_01x02_Socket, Connector_Wire:SolderWire-2sqmm_1x02_P7.8mm_D2mm_OD3.9mm_Relief, F.Cu at (201.9, 77.3)
- added J12: Conn_01x02_Socket, Connector_Wire:SolderWire-2sqmm_1x02_P7.8mm_D2mm_OD3.9mm_Relief, F.Cu at (188.4, 77.3)
- added J13: Conn_01x02_Socket, Connector_Wire:SolderWire-2sqmm_1x02_P7.8mm_D2mm_OD3.9mm_Relief, F.Cu at (174.9, 77.3)
- added J14: Conn_01x02_Socket, Connector_Wire:SolderWire-2sqmm_1x02_P7.8mm_D2mm_OD3.9mm_Relief, F.Cu at (161.4, 77.3)
- added JP7: SolderJumper_3_Open, Jumper:SolderJumper-3_P1.3mm_Open_RoundedPad1.0x1.5mm_NumberLabels, F.Cu at (106.7, 95.2)
- added JP8: SolderJumper_3_Open, Jumper:SolderJumper-3_P1.3mm_Open_RoundedPad1.0x1.5mm_NumberLabels, F.Cu at (44.3, 99.2)
- added Q1: SI2312, SI2312:SOT23, F.Cu at (24.5, 113.2)
- added Q10: SI2312, SI2312:SOT23, F.Cu at (24.5, 117.8)
- added Q11: SI2312, SI2312:SOT23, F.Cu at (28.5, 117.8)
- added Q12: SI2312, SI2312:SOT23, F.Cu at (32.5, 117.8)
- added Q13: SI2312, SI2312:SOT23, F.Cu at (36.6, 117.8)
- added Q14: SI2312, SI2312:SOT23, F.Cu at (40.6, 117.8)
- added Q15: SI2312, SI2312:SOT23, F.Cu at (44.7, 117.8)
- added Q16: SI2312, SI2312:SOT23, F.Cu at (48.7, 117.8)
- added Q17: SI2312, SI2312:SOT23, F.Cu at (52.8, 117.8)
- added Q18: SI2312, SI2312:SOT23, F.Cu at (56.8, 117.8)
- added Q19: SI2312, SI2312:SOT23, F.Cu at (24.5, 122.4)
- added Q2: SI2312, SI2312:SOT23, F.Cu at (28.5, 113.2)
- added Q20: SI2312, SI2312:SOT23, F.Cu at (28.5, 122.4)
- added Q21: SI2312, SI2312:SOT23, F.Cu at (32.5, 122.4)
- added Q22: SI2312, SI2312:SOT23, F.Cu at (36.6, 122.4)
- added Q23: SI2312, SI2312:SOT23, F.Cu at (40.6, 122.4)
- added Q24: SI2312, SI2312:SOT23, F.Cu at (44.7, 122.4)
- added Q25: SI2312, SI2312:SOT23, F.Cu at (48.7, 122.4)
- added Q26: SI2312, SI2312:SOT23, F.Cu at (52.8, 122.4)
- added Q27: SI2312, SI2312:SOT23, F.Cu at (56.8, 122.4)
- added Q28: SI2312, SI2312:SOT23, F.Cu at (24.5, 127.0)
- added Q29: SI2312, SI2312:SOT23, F.Cu at (28.5, 127.0)
- added Q3: SI2312, SI2312:SOT23, F.Cu at (32.5, 113.2)
- added Q30: SI2312, SI2312:SOT23, F.Cu at (32.5, 127.0)
- added Q31: SI2312, SI2312:SOT23, F.Cu at (36.6, 127.0)
- added Q32: SI2312, SI2312:SOT23, F.Cu at (40.6, 127.0)
- added Q33: SI2312, SI2312:SOT23, F.Cu at (44.7, 127.0)
- added Q34: SI2312, SI2312:SOT23, F.Cu at (48.7, 127.0)
- added Q35: SI2312, SI2312:SOT23, F.Cu at (52.8, 127.0)
- added Q36: SI2312, SI2312:SOT23, F.Cu at (56.8, 127.0)
- added Q37: SI2312, SI2312:SOT23, F.Cu at (24.5, 131.6)
- added Q38: SI2312, SI2312:SOT23, F.Cu at (28.5, 131.6)
- added Q39: SI2312, SI2312:SOT23, F.Cu at (32.5, 131.6)
- added Q4: SI2312, SI2312:SOT23, F.Cu at (36.6, 113.2)
- added Q40: SI2312, SI2312:SOT23, F.Cu at (36.6, 131.6)
- added Q41: SI2312, SI2312:SOT23, F.Cu at (40.6, 131.6)
- added Q42: SI2312, SI2312:SOT23, F.Cu at (44.7, 131.6)
- added Q43: SI2312, SI2312:SOT23, F.Cu at (48.7, 131.6)
- added Q44: SI2312, SI2312:SOT23, F.Cu at (52.8, 131.6)
- added Q45: SI2312, SI2312:SOT23, F.Cu at (56.8, 131.6)
- added Q46: SI2312, SI2312:SOT23, F.Cu at (24.5, 136.2)
- added Q47: SI2312, SI2312:SOT23, F.Cu at (28.5, 136.2)
- added Q48: SI2312, SI2312:SOT23, F.Cu at (32.5, 136.2)
- added Q49: SI2312, SI2312:SOT23, F.Cu at (24.5, 142.8)
- added Q5: SI2312, SI2312:SOT23, F.Cu at (40.6, 113.2)
- added Q50: SI2312, SI2312:SOT23, F.Cu at (28.5, 142.8)
- added Q51: SI2312, SI2312:SOT23, F.Cu at (32.5, 142.8)
- added Q52: SI2312, SI2312:SOT23, F.Cu at (36.6, 142.8)
- added Q6: SI2312, SI2312:SOT23, F.Cu at (44.7, 113.2)
- added Q7: SI2312, SI2312:SOT23, F.Cu at (48.7, 113.2)
- added Q8: SI2312, SI2312:SOT23, F.Cu at (52.8, 113.2)
- added Q9: SI2312, SI2312:SOT23, F.Cu at (56.8, 113.2)
- added R10: R, Resistor_SMD:R_0805_2012Metric_Pad1.20x1.40mm_HandSolder, F.Cu at (34.3, 97.1)
- added R11: R, Resistor_SMD:R_0805_2012Metric_Pad1.20x1.40mm_HandSolder, F.Cu at (34.3, 100.0)
- added R12: R, Resistor_SMD:R_0805_2012Metric_Pad1.20x1.40mm_HandSolder, F.Cu at (39.1, 88.2)
- added R13: R, Resistor_SMD:R_0805_2012Metric_Pad1.20x1.40mm_HandSolder, F.Cu at (39.1, 91.2)
- added R14: R, Resistor_SMD:R_0805_2012Metric_Pad1.20x1.40mm_HandSolder, F.Cu at (39.1, 94.2)
- added R15: R, Resistor_SMD:R_0805_2012Metric_Pad1.20x1.40mm_HandSolder, F.Cu at (39.1, 97.1)
- added R2: R, Resistor_SMD:R_0805_2012Metric_Pad1.20x1.40mm_HandSolder, F.Cu at (29.6, 88.2)
- added R3: R, Resistor_SMD:R_0805_2012Metric_Pad1.20x1.40mm_HandSolder, F.Cu at (29.6, 91.2)
- added R4: R, Resistor_SMD:R_0805_2012Metric_Pad1.20x1.40mm_HandSolder, F.Cu at (29.6, 94.2)
- added R5: R, Resistor_SMD:R_0805_2012Metric_Pad1.20x1.40mm_HandSolder, F.Cu at (29.6, 97.1)
- added R6: R, Resistor_SMD:R_0805_2012Metric_Pad1.20x1.40mm_HandSolder, F.Cu at (29.6, 100.0)
- added R7: R, Resistor_SMD:R_0805_2012Metric_Pad1.20x1.40mm_HandSolder, F.Cu at (34.3, 88.2)
- added R8: R, Resistor_SMD:R_0805_2012Metric_Pad1.20x1.40mm_HandSolder, F.Cu at (34.3, 91.2)
- added R9: R, Resistor_SMD:R_0805_2012Metric_Pad1.20x1.40mm_HandSolder, F.Cu at (34.3, 94.2)
- added U14: BME280, Package_LGA:Bosch_LGA-8_2.5x2.5mm_P0.65mm_ClockwisePinNumbering, F.Cu at (63.1, 81.2)
- added U4: ACS712xLCTR-20A, Package_SO:SOIC-8_3.9x4.9mm_P1.27mm, F.Cu at (23.0, 54.9)
- added Y1: 32.786KHz, Crystal:Crystal_DS26_D2.0mm_L6.0mm_Horizontal, F.Cu at (62.2, 69.7)
- added Y2: 25MHz, Crystal:Crystal_SMD_HC49-SD, F.Cu at (58.6, 98.2)
- added Y3: 25MHz, Crystal:Crystal_SMD_HC49-SD, F.Cu at (75.1, 90.2)
- added Y4: 32.786KHz, Crystal:Crystal_DS26_D2.0mm_L6.0mm_Horizontal, F.Cu at (83.7, 88.0)
- J3, J4: value Conn_01x02_Socket -> Conn_01x03_Socket; footprint Connector_Wire:SolderWire-2sqmm_1x02_P7.8mm_D2mm_OD3.9mm_Relief -> Connector_JST:JST_XH_B3B-XH-A_1x03_P2.50mm_Vertical
- J5, J6: footprint Connector_Wire:SolderWire-2sqmm_1x02_P7.8mm_D2mm_OD3.9mm_Relief -> Connector_JST:JST_XH_B2B-XH-A_1x02_P2.50mm_Vertical
- J8: value Conn_01x03_Socket -> Conn_01x05_Socket; footprint Connector_Wire:SolderWire-0.5sqmm_1x03_P4.6mm_D0.9mm_OD2.1mm_Relief -> Connector_Wire:SolderWire-0.5sqmm_1x05_P4.8mm_D0.9mm_OD2.3mm_Relief
- J9: value Conn_01x03_Socket -> Conn_01x02_Socket; footprint Connector_Wire:SolderWire-0.5sqmm_1x03_P4.6mm_D0.9mm_OD2.1mm_Relief -> Connector_Wire:SolderWire-2sqmm_1x02_P7.8mm_D2mm_OD3.9mm_Relief
- moved J1 197.4 mm to (242.4, 77.3), turned to 180 degrees
- moved JP1 178.5 mm to (44.3, 88.5)
- moved JP2 178.5 mm to (44.3, 92.1)
- moved JP3 178.5 mm to (44.3, 95.7)
- moved J2 127.5 mm to (228.9, 77.3), turned to 180 degrees
- moved U6 102.8 mm to (70.5, 54.4)
- moved U10 90.1 mm to (23.0, 81.2)
- moved U11 90.1 mm to (23.0, 87.8)
- moved U7 90.1 mm to (23.0, 61.5)
- moved U8 90.1 mm to (23.0, 68.1)
- moved U9 90.1 mm to (23.0, 74.7)
- moved U5 90.1 mm to (29.9, 54.4)
- moved JP4 81.1 mm to (106.7, 84.6)
- moved JP5 81.1 mm to (106.7, 88.2)
- moved JP6 81.1 mm to (106.7, 91.7)
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Connections:
- J2 pad 1: MOTOR1IN -> Net-(J2-Pin_1)
- J2 pad 2: MOTOR1OUT -> Net-(J2-Pin_2)
- J3 pad 1: MOTOR2IN -> +5V
- J3 pad 2: MOTOR2OUT -> Net-(J3-Pin_2)
- J4 pad 1: MOTOR3IN -> +5V
- J4 pad 2: MOTOR3OUT -> Net-(J4-Pin_2)
- J5 pad 1: MOTOR4IN -> Net-(J5-Pin_1)
- J5 pad 2: MOTOR4OUT -> GND
- J6 pad 1: MOTOR5IN -> Net-(J6-Pin_1)
- J6 pad 2: MOTOR5OUT -> GND
- J8 pad 1: Net-(J8-Pin_1) -> GND
- JP1 pad 1: Net-(J8-Pin_3) -> Net-(J8-Pin_5)
- JP2 pad 1: Net-(J8-Pin_2) -> Net-(J8-Pin_4)
- JP3 pad 1: Net-(J8-Pin_1) -> Net-(J8-Pin_3)
- JP4 pad 1: Net-(J9-Pin_1) -> Net-(J10-Pin_3)
- JP4 pad 2: unconnected-(JP4-C-Pad2) -> Net-(JP4-C)
- JP4 pad 3: unconnected-(JP4-B-Pad3) -> Net-(JP4-B)
- JP5 pad 1: Net-(J9-Pin_2) -> Net-(J10-Pin_4)
- JP5 pad 2: unconnected-(JP5-C-Pad2) -> Net-(JP5-C)
- JP5 pad 3: unconnected-(JP5-B-Pad3) -> Net-(JP5-B)
- JP6 pad 1: Net-(J9-Pin_3) -> Net-(J10-Pin_5)
- JP6 pad 2: unconnected-(JP6-C-Pad2) -> Net-(JP6-C)
- JP6 pad 3: unconnected-(JP6-B-Pad3) -> Net-(JP6-B)
- U10 pad 1: MOTOR6a -> MOTOR6IN
- U10 pad 2: MOTOR6a -> MOTOR6IN
- U10 pad 3: MOTOR6IN -> GND
- U10 pad 4: MOTOR6IN -> GND
- U10 pad 6: unconnected-(U10-FILTER-Pad6) -> Net-(U10-FILTER)
- U11 pad 1: MOTOR1a -> MOTOR1IN
- U11 pad 2: MOTOR1a -> MOTOR1IN
- U11 pad 3: MOTOR1IN -> GND
- U11 pad 4: MOTOR1IN -> GND
- U11 pad 6: unconnected-(U11-FILTER-Pad6) -> Net-(U11-FILTER)
- U12 pad 10: unconnected-(U12-PC2-Pad10) -> MOTOR2a
- U12 pad 11: unconnected-(U12-PC3-Pad11) -> MOTOR2b
- U12 pad 14: Net-(U12-PA0) -> unconnected-(U12-PA0-Pad14)
- U12 pad 15: Net-(U12-PA1) -> unconnected-(U12-PA1-Pad15)
- U12 pad 16: Net-(U12-PA2) -> unconnected-(U12-PA2-Pad16)
- U12 pad 21: Net-(U12-PA5) -> Net-(JP6-C)
- U12 pad 22: unconnected-(U12-PA6-Pad22) -> Net-(JP5-C)
- U12 pad 23: unconnected-(U12-PA7-Pad23) -> Net-(JP4-C)
- U12 pad 24: unconnected-(U12-PC4-Pad24) -> MOTOR3a
- U12 pad 25: unconnected-(U12-PC5-Pad25) -> MOTOR3b
- U12 pad 26: unconnected-(U12-PB0-Pad26) -> PWM1
- U12 pad 27: unconnected-(U12-PB1-Pad27) -> PWM2
- U12 pad 28: unconnected-(U12-PB2-Pad28) -> PWM3
- U12 pad 3: unconnected-(U12-PC14-Pad3) -> Net-(U12-PC14)
- U12 pad 37: unconnected-(U12-PC6-Pad37) -> MOTOR4a
- U12 pad 38: unconnected-(U12-PC7-Pad38) -> MOTOR4b
- U12 pad 39: unconnected-(U12-PC8-Pad39) -> MOTOR5a
- U12 pad 4: unconnected-(U12-PC15-Pad4) -> Net-(U12-PC15)
- U12 pad 40: unconnected-(U12-PC9-Pad40) -> MOTOR5b
- U12 pad 5: unconnected-(U12-PH0-Pad5) -> Net-(U12-PH0)
- U12 pad 51: unconnected-(U12-PC10-Pad51) -> MOTOR6a
- U12 pad 52: unconnected-(U12-PC11-Pad52) -> MOTOR6b
- U12 pad 55: unconnected-(U12-PB3-Pad55) -> PWM4
- U12 pad 6: unconnected-(U12-PH1-Pad6) -> Net-(U12-PH1)
- U12 pad 8: unconnected-(U12-PC0-Pad8) -> MOTOR1a
- U12 pad 9: unconnected-(U12-PC1-Pad9) -> MOTOR1b
- U13 pad 20: Net-(U13-PB2) -> Net-(JP8-C)
- U3 pad 1: unconnected-(U3-IN-Pad1) -> VCC
- U5 pad 4: Net-(U13-PB2) -> Net-(JP8-B)
- U6 pad 1: unconnected-(U6-GND-Pad1) -> GND
- U6 pad 2: unconnected-(U6-VCC-Pad2) -> +3.3V
- U6 pad 3: unconnected-(U6-CE-Pad3) -> Net-(U12-PA3)
- U6 pad 4: unconnected-(U6-~{CSN}-Pad4) -> Net-(JP7-B)
- U6 pad 5: unconnected-(U6-SCK-Pad5) -> Net-(JP6-B)
- U6 pad 6: unconnected-(U6-MOSI-Pad6) -> Net-(JP4-B)
- U6 pad 7: unconnected-(U6-MISO-Pad7) -> Net-(JP5-B)
- U7 pad 1: MOTOR3a -> MOTOR3IN
- U7 pad 2: MOTOR3a -> MOTOR3IN
- U7 pad 3: MOTOR3IN -> GND
- U7 pad 4: MOTOR3IN -> GND
- U7 pad 6: unconnected-(U7-FILTER-Pad6) -> Net-(U7-FILTER)
- U8 pad 1: MOTOR4a -> MOTOR4IN
- U8 pad 2: MOTOR4a -> MOTOR4IN
- U8 pad 3: MOTOR4IN -> GND
- U8 pad 4: MOTOR4IN -> GND
- U8 pad 6: unconnected-(U8-FILTER-Pad6) -> Net-(U8-FILTER)
- U9 pad 1: MOTOR5a -> MOTOR56IN
- U9 pad 2: MOTOR5a -> MOTOR56IN
- U9 pad 3: MOTOR56IN -> GND
- U9 pad 4: MOTOR56IN -> GND
- U9 pad 6: unconnected-(U9-FILTER-Pad6) -> Net-(U9-FILTER)
Routing:
- net VCC: track 11.9 -> 0.00 mm
- net GND: track 10.8 -> 0.00 mm
- net +3.3V: track 6.30 -> 0.00 mm
- net +5V: track 4.93 -> 0.00 mm
Other:
- board outline added: 100 x 100 mm

Commit message: adding completation on schematic, working on board
need to add SWD Debug as input for programing
Parts:
- added C15: 12,5pF, Capacitor_SMD:C_0805_2012Metric_Pad1.18x1.45mm_HandSolder, F.Cu at (62.5, 41.4)
- added C16: 12,5pF, Capacitor_SMD:C_0805_2012Metric_Pad1.18x1.45mm_HandSolder, F.Cu at (51.0, 51.0)
- added H1: MountingHole_Pad, MountingHole:MountingHole_3.5mm_Pad_Via, F.Cu at (245.0, 55.0)
- added H2: MountingHole_Pad, MountingHole:MountingHole_3.5mm_Pad_Via, F.Cu at (155.0, 55.0)
- added H3: MountingHole_Pad, MountingHole:MountingHole_3.5mm_Pad_Via, F.Cu at (245.0, 145.0)
- added H4: MountingHole_Pad, MountingHole:MountingHole_3.5mm_Pad_Via, F.Cu at (155.0, 145.0)
- added J14: Conn_01x02_Socket, Connector_Wire:SolderWire-2sqmm_1x02_P7.8mm_D2mm_OD3.9mm, F.Cu at (198.0, 53.0)
- added R10: 10K, Resistor_SMD:R_0805_2012Metric_Pad1.20x1.40mm_HandSolder, F.Cu at (44.8, 39.2)
- added R11: 10K, Resistor_SMD:R_0805_2012Metric_Pad1.20x1.40mm_HandSolder, F.Cu at (44.8, 42.1)
- added R12: 10K, Resistor_SMD:R_0805_2012Metric_Pad1.20x1.40mm_HandSolder, F.Cu at (44.8, 45.1)
- added R13: 10K, Resistor_SMD:R_0805_2012Metric_Pad1.20x1.40mm_HandSolder, F.Cu at (44.8, 48.0)
- added R14: 10K, Resistor_SMD:R_0805_2012Metric_Pad1.20x1.40mm_HandSolder, F.Cu at (49.6, 36.2)
- added R15: 10K, Resistor_SMD:R_0805_2012Metric_Pad1.20x1.40mm_HandSolder, F.Cu at (57.7, 41.4)
- added R16: 10K, Resistor_SMD:R_0805_2012Metric_Pad1.20x1.40mm_HandSolder, F.Cu at (57.7, 44.3)
- added R17: 10K, Resistor_SMD:R_0805_2012Metric_Pad1.20x1.40mm_HandSolder, F.Cu at (49.6, 39.2)
- added R18: 10K, Resistor_SMD:R_0805_2012Metric_Pad1.20x1.40mm_HandSolder, F.Cu at (49.6, 42.1)
- added R4: 10K, Resistor_SMD:R_0805_2012Metric_Pad1.20x1.40mm_HandSolder, F.Cu at (40.1, 36.2)
- added R5: 10K, Resistor_SMD:R_0805_2012Metric_Pad1.20x1.40mm_HandSolder, F.Cu at (40.1, 39.2)
- added R6: 10K, Resistor_SMD:R_0805_2012Metric_Pad1.20x1.40mm_HandSolder, F.Cu at (40.1, 42.1)
- added R7: 10K, Resistor_SMD:R_0805_2012Metric_Pad1.20x1.40mm_HandSolder, F.Cu at (40.1, 45.1)
- added R8: 10K, Resistor_SMD:R_0805_2012Metric_Pad1.20x1.40mm_HandSolder, F.Cu at (40.1, 48.0)
- added R9: 10K, Resistor_SMD:R_0805_2012Metric_Pad1.20x1.40mm_HandSolder, F.Cu at (44.8, 36.2)
- added SW1: SW_Push, Button_Switch_SMD:SW_SPST_CK_RS282G05A3, F.Cu at (195.2, 67.0)
- added SW2: SW_Push, Button_Switch_SMD:SW_SPST_CK_RS282G05A3, F.Cu at (43.1, 52.1)
- C1: renamed from C9; moved to B.Cu
- C2: renamed from C10; moved to B.Cu
- C3: renamed from C7; moved to B.Cu
- C4: renamed from C8; moved to B.Cu
- J1, J9: footprint Connector_Wire:SolderWire-2sqmm_1x02_P7.8mm_D2mm_OD3.9mm_Relief -> Connector_Wire:SolderWire-2sqmm_1x02_P7.8mm_D2mm_OD3.9mm
- J10: renamed from J11; footprint Connector_Wire:SolderWire-2sqmm_1x02_P7.8mm_D2mm_OD3.9mm_Relief -> Connector_Wire:SolderWire-2sqmm_1x02_P7.8mm_D2mm_OD3.9mm
- J11: renamed from J12; footprint Connector_Wire:SolderWire-2sqmm_1x02_P7.8mm_D2mm_OD3.9mm_Relief -> Connector_Wire:SolderWire-2sqmm_1x02_P7.8mm_D2mm_OD3.9mm
- J12: renamed from J13; footprint Connector_Wire:SolderWire-2sqmm_1x02_P7.8mm_D2mm_OD3.9mm_Relief -> Connector_Wire:SolderWire-2sqmm_1x02_P7.8mm_D2mm_OD3.9mm
- J13: renamed from J14; footprint Connector_Wire:SolderWire-2sqmm_1x02_P7.8mm_D2mm_OD3.9mm_Relief -> Connector_Wire:SolderWire-2sqmm_1x02_P7.8mm_D2mm_OD3.9mm
- J8: renamed from J2; footprint Connector_Wire:SolderWire-2sqmm_1x02_P7.8mm_D2mm_OD3.9mm_Relief -> Connector_Wire:SolderWire-2sqmm_1x02_P7.8mm_D2mm_OD3.9mm
- JP1, JP2, JP3, Y1, Y2: moved to B.Cu
- JP4: renamed from JP8; moved to B.Cu
- R1: renamed from R14; value R -> 10K
- R2: renamed from R15; value R -> 10K
- R3: renamed from R2; value R -> 10K
- U5: renamed from U13; moved to B.Cu
- moved U4 206.1 mm to (233.5, 86.4)
- moved JP1 187.5 mm to (230.0, 63.0), turned to -90 degrees
- moved JP3 187.1 mm to (230.0, 73.0), turned to -90 degrees
- moved JP2 185.3 mm to (228.0, 68.0), turned to -90 degrees
- moved JP4 185.0 mm to (228.0, 78.0), turned to -90 degrees
- moved C12 181.3 mm to (215.2, 130.2), turned to -90 degrees
- moved C11 179.2 mm to (215.2, 136.0), turned to -90 degrees
- moved Q2 173.7 mm to (198.1, 140.4), turned to -90 degrees
- moved Q1 173.6 mm to (202.1, 140.4), turned to -90 degrees
- moved U12 169.9 mm to (233.5, 102.4)
- moved C14 163.8 mm to (203.2, 132.2)
- moved C1 161.7 mm to (220.0, 86.0), turned to -90 degrees
- moved C13 160.3 mm to (203.2, 128.5)
- moved C2 158.6 mm to (217.0, 87.0), turned to 180 degrees
- moved Q4 157.6 mm to (190.1, 140.4), turned to -90 degrees
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- renumbered C6 to C10, C12 to C11, C11 to C12, C14 to C13, C13 to C14, C1 to C5, C2 to C6, C3 to C7, C4 to C8, C5 to C9, J8 to J2, J10 to J3, J3 to J4, J4 to J5, J5 to J6, J6 to J7, JP6 to JP5, JP5 to JP6, JP4 to JP7, JP7 to JP8, Q50 to Q1, Q18 to Q10, Q2 to Q11, Q6 to Q12, Q11 to Q13, Q12 to Q14, Q19 to Q15, Q20 to Q16, Q3 to Q17, Q7 to Q18, Q13 to Q19, Q49 to Q2, Q14 to Q20, Q4 to Q23, Q8 to Q24, Q15 to Q25, Q16 to Q26, Q23 to Q27, Q24 to Q28, Q25 to Q29, Q52 to Q3, Q26 to Q30, Q27 to Q31, Q28 to Q32, Q29 to Q33, Q30 to Q34, Q31 to Q35, Q32 to Q36, Q33 to Q37, Q34 to Q38, Q35 to Q39, Q51 to Q4, Q36 to Q40, Q37 to Q41, Q38 to Q42, Q39 to Q43, Q40 to Q44, Q41 to Q45, Q42 to Q46, Q43 to Q47, Q44 to Q48, Q45 to Q49, Q1 to Q5, Q46 to Q50, Q47 to Q51, Q48 to Q52, Q5 to Q6, Q9 to Q7, Q10 to Q8, Q17 to Q9, R9 to R10, R10 to R11, R11 to R12, R12 to R13, R13 to R14, R3 to R4, R4 to R5, R5 to R6, R6 to R7, R7 to R8, R8 to R9, U3 to U1, U9 to U10, U10 to U11, U6 to U12, U12 to U13, U1 to U2, U14 to U3, U5 to U4, U11 to U6, U4 to U7, U7 to U8, U8 to U9
Connections:
- J10 pad 1: MOTOR3b -> Net-(J10-Pin_1)
- Q10 pad 1: MOTOR3b -> MOTOR1b
- Q13 pad 1: MOTOR2a -> MOTOR1a
- Q14 pad 1: MOTOR2b -> MOTOR1b
- Q15 pad 1: MOTOR3a -> MOTOR1a
- Q16 pad 1: MOTOR3b -> MOTOR1b
- Q19 pad 1: MOTOR2b -> MOTOR1b
- Q20 pad 1: MOTOR2a -> MOTOR1a
- Q21 pad 1: Net-(Q21-Pad1) -> MOTOR1b
- Q21 pad 2: MOTOR3b -> Net-(J10-Pin_1)
- Q22 pad 1: MOTOR3a -> MOTOR1a
- Q22 pad 3: MOTOR3b -> Net-(J10-Pin_1)
- Q25 pad 1: MOTOR2b -> MOTOR1b
- Q26 pad 1: MOTOR2a -> MOTOR1a
- Q27 pad 1: Net-(Q21-Pad1) -> MOTOR1b
- Q27 pad 2: MOTOR3b -> Net-(J10-Pin_1)
- Q28 pad 1: MOTOR3a -> MOTOR1a
- Q28 pad 3: MOTOR3b -> Net-(J10-Pin_1)
- Q31 pad 1: MOTOR5a -> MOTOR4a
- Q32 pad 1: MOTOR5b -> MOTOR4b
- Q33 pad 1: MOTOR6a -> MOTOR4a
- Q34 pad 1: MOTOR6b -> MOTOR4b
- Q37 pad 1: MOTOR5a -> MOTOR4a
- Q38 pad 1: MOTOR5b -> MOTOR4b
- Q39 pad 1: MOTOR6a -> MOTOR4a
- Q40 pad 1: MOTOR6b -> MOTOR4b
- Q43 pad 1: MOTOR5b -> MOTOR4b
- Q44 pad 1: MOTOR5a -> MOTOR4a
- Q45 pad 1: MOTOR6b -> MOTOR4b
- Q46 pad 1: MOTOR6a -> MOTOR4a
- Q49 pad 1: MOTOR5b -> MOTOR4b
- Q50 pad 1: MOTOR5a -> MOTOR4a
- Q51 pad 1: MOTOR6b -> MOTOR4b
- Q52 pad 1: MOTOR6a -> MOTOR4a
- Q7 pad 1: MOTOR2a -> MOTOR1a
- Q8 pad 1: MOTOR2b -> MOTOR1b
- Q9 pad 1: MOTOR3a -> MOTOR1a
- U13 pad 1: unconnected-(U12-VBAT-Pad1) -> +3.3V
- U13 pad 12: unconnected-(U12-VSSA-Pad12) -> GND
- U13 pad 13: unconnected-(U12-VDDA-Pad13) -> +3.3V
- U13 pad 18: Net-(U12-VSS-Pad18) -> GND
- U13 pad 19: unconnected-(U12-VDD-Pad19) -> +3.3V
- U13 pad 24: MOTOR3a -> unconnected-(U13-PC4-Pad24)
- U13 pad 25: MOTOR3b -> unconnected-(U13-PC5-Pad25)
- U13 pad 31: Net-(U12-VSS-Pad18) -> GND
- U13 pad 32: unconnected-(U12-VDD-Pad32) -> +3.3V
- U13 pad 37: MOTOR4a -> unconnected-(U13-PC6-Pad37)
- U13 pad 38: MOTOR4b -> unconnected-(U13-PC7-Pad38)
- U13 pad 39: MOTOR5a -> unconnected-(U13-PC8-Pad39)
- U13 pad 40: MOTOR5b -> unconnected-(U13-PC9-Pad40)
- U13 pad 47: Net-(U12-VSS-Pad18) -> GND
- U13 pad 48: unconnected-(U12-VDD-Pad48) -> +3.3V
- U13 pad 51: MOTOR6a -> unconnected-(U13-PC10-Pad51)
- U13 pad 52: MOTOR6b -> unconnected-(U13-PC11-Pad52)
- U13 pad 60: unconnected-(U12-BOOT0-Pad60) -> Net-(U13-BOOT0)
- U13 pad 63: Net-(U12-VSS-Pad18) -> GND
- U13 pad 64: unconnected-(U12-VDD-Pad64) -> +3.3V
- U13 pad 7: unconnected-(U12-NRST-Pad7) -> Net-(U13-NRST)
- U5 pad 44: unconnected-(U13-BOOT0-Pad44) -> Net-(U5-BOOT0)
- U5 pad 7: unconnected-(U13-NRST-Pad7) -> Net-(U5-NRST)
Routing:
- net GND: track 0.00 -> 62.5 mm
- net Net-(U12-CE): track 0.00 -> 61.7 mm
- net PWM3: track 0.00 -> 39.5 mm, vias 0 -> 2
- net PWM2: track 0.00 -> 36.8 mm, vias 0 -> 2
- net Net-(JP8-B): track 0.00 -> 35.1 mm
- net PWM1: track 0.00 -> 34.9 mm, vias 0 -> 2
- net Net-(JP1-B): track 0.00 -> 33.6 mm
- net Net-(JP2-B): track 0.00 -> 33.3 mm
- net Net-(JP7-B): track 0.00 -> 25.7 mm
- net Net-(JP4-C): track 0.00 -> 23.0 mm
- net PWM4: track 0.00 -> 22.6 mm
- net Net-(JP3-B): track 0.00 -> 22.0 mm
- net Net-(JP1-C): track 0.00 -> 21.2 mm, vias 0 -> 2
- net Net-(JP7-C): track 0.00 -> 20.4 mm, vias 0 -> 2
- net Net-(JP6-B): track 0.00 -> 20.3 mm
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Other:
- copper layers 2 -> 4

Commit message: .
Parts:
- removed the R10 at (44.8, 39.2)
- removed the R10 at (34.3, 94.2)
- removed the R11 at (34.3, 97.1)
- removed the R11 at (44.8, 42.1)
- removed the R12 at (34.3, 100.0)
- removed the R12 at (44.8, 45.1)
- removed the R13 at (44.8, 48.0)
- removed the R13 at (39.1, 88.2)
- removed the R14 at (49.6, 36.2)
- removed the R14 at (39.1, 91.2)
- removed the R4 at (40.1, 36.2)
- removed the R4 at (29.6, 91.2)
- removed the R5 at (29.6, 94.2)
- removed the R5 at (40.1, 39.2)
- removed the R6 at (40.1, 42.1)
- removed the R6 at (29.6, 97.1)
- removed the R7 at (40.1, 45.1)
- removed the R7 at (29.6, 100.0)
- removed the R8 at (40.1, 48.0)
- removed the R8 at (34.3, 88.2)
- removed the R9 at (44.8, 36.2)
- removed the R9 at (34.3, 91.2)
- added R10: 10K, Resistor_SMD:R_0805_2012Metric_Pad1.20x1.40mm_HandSolder, F.Cu at (120.2, 88.2)
- added R11: 10K, Resistor_SMD:R_0805_2012Metric_Pad1.20x1.40mm_HandSolder, F.Cu at (120.2, 91.1)
- added R12: 10K, Resistor_SMD:R_0805_2012Metric_Pad1.20x1.40mm_HandSolder, F.Cu at (162.0, 79.8)
- added R13: 10K, Resistor_SMD:R_0805_2012Metric_Pad1.20x1.40mm_HandSolder, F.Cu at (125.0, 85.2)
- added R14: 10K, Resistor_SMD:R_0805_2012Metric_Pad1.20x1.40mm_HandSolder, F.Cu at (125.0, 88.2)
- added R4: 10K, Resistor_SMD:R_0805_2012Metric_Pad1.20x1.40mm_HandSolder, F.Cu at (184.0, 108.2)
- added R5: 10K, Resistor_SMD:R_0805_2012Metric_Pad1.20x1.40mm_HandSolder, F.Cu at (174.2, 106.0)
- added R6: 10K, Resistor_SMD:R_0805_2012Metric_Pad1.20x1.40mm_HandSolder, F.Cu at (172.0, 109.0)
- added R7: 10K, Resistor_SMD:R_0805_2012Metric_Pad1.20x1.40mm_HandSolder, F.Cu at (157.0, 105.8)
- added R8: 10K, Resistor_SMD:R_0805_2012Metric_Pad1.20x1.40mm_HandSolder, F.Cu at (155.5, 108.8)
- added R9: 10K, Resistor_SMD:R_0805_2012Metric_Pad1.20x1.40mm_HandSolder, F.Cu at (154.0, 77.8)
- C16, R18: moved to B.Cu
- moved R15 183.7 mm to (218.5, 130.2), turned to -90 degrees
- moved R1 174.3 mm to (211.8, 70.2)
- moved R2 171.6 mm to (208.8, 71.5), turned to 90 degrees
- moved R18 171.2 mm to (217.8, 74.2), turned to 90 degrees
- moved SW2 168.9 mm to (211.5, 66.0), turned to 180 degrees
- moved Q5 166.4 mm to (190.0, 130.0), turned to 180 degrees
- moved U6 166.2 mm to (187.8, 109.8), turned to 90 degrees
- moved Q33 164.2 mm to (190.5, 100.2), turned to 180 degrees
- moved U7 163.4 mm to (176.5, 110.8), turned to 90 degrees
- moved Q34 162.3 mm to (190.5, 89.8), turned to 180 degrees
- moved U11 162.0 mm to (185.0, 82.5), turned to 90 degrees
- moved Q51 159.1 mm to (183.5, 100.2), turned to 180 degrees
- moved Q11 158.9 mm to (186.5, 130.0), turned to 180 degrees
- moved R16 158.8 mm to (204.5, 105.0)
- moved C5 158.6 mm to (189.7, 104.8)
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Connections:
- C6 pad 1: unconnected-(C6-Pad1) -> Net-(U7-FILTER)
- U10 pad 1: MOTOR56IN -> MOTOR5IN
- U10 pad 2: MOTOR56IN -> MOTOR5IN
- U10 pad 8: +3.3V -> +5V
- U11 pad 8: +3.3V -> +5V
- U6 pad 8: +3.3V -> +5V
- U7 pad 6: unconnected-(U7-FILTER-Pad6) -> Net-(U7-FILTER)
- U7 pad 8: +3.3V -> +5V
- U8 pad 8: +3.3V -> +5V
- U9 pad 8: +3.3V -> +5V
Routing:
- net GND: track 62.5 -> 338.8 mm, vias 0 -> 6
- net VCC: track 0.00 -> 184.8 mm
- net +5V: track 12.0 -> 172.8 mm, vias 0 -> 6
- net MOTOR1b: track 0.00 -> 87.7 mm, vias 0 -> 12
- net MOTOR1a: track 0.00 -> 85.2 mm, vias 0 -> 12
- net Net-(U5-PA2): track 0.00 -> 71.9 mm, vias 0 -> 2
- net Net-(U5-PA1): track 0.00 -> 60.0 mm, vias 0 -> 2
- net +3.3V: track 2.72 -> 57.6 mm, vias 0 -> 2
- net Net-(U5-PA0): track 0.00 -> 48.4 mm, vias 0 -> 2
- net MOTOR1IN: track 0.00 -> 31.6 mm
- net MOTOR3IN: track 0.00 -> 29.6 mm
- net MOTOR2IN: track 0.00 -> 24.4 mm
- net Net-(J10-Pin_1): track 0.00 -> 21.6 mm
- net MOTOR4IN: track 0.00 -> 20.7 mm
- net MOTOR6IN: track 0.00 -> 20.6 mm
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
Commit message: .
Parts:
- C15: moved to B.Cu
- moved R17 81.0 mm to (204.8, 77.2), turned to 90 degrees
- moved C15 65.1 mm to (207.0, 123.2), turned to -90 degrees
- moved R13 58.2 mm to (182.8, 77.8), turned to 180 degrees
- moved R14 56.7 mm to (181.2, 80.8), turned to -90 degrees
- moved R11 49.8 mm to (168.2, 77.8), turned to 180 degrees
- moved R10 32.6 mm to (152.0, 80.8), turned to -90 degrees
- moved R12 4.85 mm to (166.8, 80.8), turned to -90 degrees
- moved U2 0.75 mm to (156.0, 65.7)
- moved C16 0.25 mm to (204.5, 77.2)
Connections:
- Q29 pad 1: MOTOR4a -> MOTOR2a
- Q30 pad 1: MOTOR4b -> MOTOR2b
- Q31 pad 1: MOTOR4a -> MOTOR2a
- Q32 pad 1: MOTOR4b -> MOTOR2b
- Q33 pad 1: MOTOR4a -> MOTOR2a
- Q34 pad 1: MOTOR4b -> MOTOR2b
- Q35 pad 1: MOTOR4a -> MOTOR2a
- Q36 pad 1: MOTOR4b -> MOTOR2b
- Q37 pad 1: MOTOR4a -> MOTOR2a
- Q38 pad 1: MOTOR4b -> MOTOR2b
- Q39 pad 1: MOTOR4a -> MOTOR2a
- Q40 pad 1: MOTOR4b -> MOTOR2b
- Q41 pad 1: MOTOR4b -> MOTOR2b
- Q42 pad 1: MOTOR4a -> MOTOR2a
- Q43 pad 1: MOTOR4b -> MOTOR2b
- Q44 pad 1: MOTOR4a -> MOTOR2a
- Q45 pad 1: MOTOR4b -> MOTOR2b
- Q46 pad 1: MOTOR4a -> MOTOR2a
- Q47 pad 1: MOTOR4b -> MOTOR2b
- Q48 pad 1: MOTOR4a -> MOTOR2a
- Q49 pad 1: MOTOR4b -> MOTOR2b
- Q50 pad 1: MOTOR4a -> MOTOR2a
- Q51 pad 1: MOTOR4b -> MOTOR2b
- Q52 pad 1: MOTOR4a -> MOTOR2a
Routing:
- net GND: track 338.8 -> 802.8 mm, vias 6 -> 12
- net +3.3V: track 57.6 -> 229.0 mm, vias 2 -> 13
- net MOTOR2b: track 0.00 -> 137.6 mm, vias 0 -> 13
- net MOTOR2a: track 0.00 -> 137.5 mm, vias 0 -> 2
- net Net-(U5-PA3): track 0.00 -> 61.8 mm, vias 0 -> 2
- net +5V: track 172.8 -> 233.8 mm, vias 6 -> 7
- net Net-(U5-PA4): track 0.00 -> 47.0 mm, vias 0 -> 2
- net Net-(U4-CE): track 0.00 -> 36.4 mm, vias 0 -> 1
- net Net-(U5-PA5): track 0.00 -> 33.7 mm, vias 0 -> 2
- net MOTOR1a: track 85.2 -> 105.9 mm, vias 12 -> 13
- net MOTOR1b: track 87.7 -> 107.5 mm, vias 12 -> 13
- net VCC: track 184.8 -> 202.9 mm
- net Net-(U11-VIOUT): track 0.00 -> 2.53 mm
- net Net-(U10-VIOUT): track 0.00 -> 2.53 mm
- net Net-(U9-VIOUT): track 0.00 -> 2.43 mm
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
Commit message: .
Connections:
- U13 pad 10: MOTOR2a -> unconnected-(U13-PC2-Pad10)
- U13 pad 11: MOTOR2b -> unconnected-(U13-PC3-Pad11)
- U13 pad 26: PWM1 -> unconnected-(U13-PB0-Pad26)
- U13 pad 27: PWM2 -> unconnected-(U13-PB1-Pad27)
- U13 pad 28: PWM3 -> unconnected-(U13-PB2-Pad28)
- U13 pad 37: unconnected-(U13-PC6-Pad37) -> MOTOR1a
- U13 pad 38: unconnected-(U13-PC7-Pad38) -> MOTOR1b
- U13 pad 39: unconnected-(U13-PC8-Pad39) -> MOTOR2a
- U13 pad 40: unconnected-(U13-PC9-Pad40) -> MOTOR2b
- U13 pad 41: unconnected-(U13-PA8-Pad41) -> PWM1
- U13 pad 42: unconnected-(U13-PA9-Pad42) -> PWM2
- U13 pad 43: unconnected-(U13-PA10-Pad43) -> PWM3
- U13 pad 44: unconnected-(U13-PA11-Pad44) -> PWM4
- U13 pad 55: PWM4 -> unconnected-(U13-PB3-Pad55)
- U13 pad 8: MOTOR1a -> unconnected-(U13-PC0-Pad8)
- U13 pad 9: MOTOR1b -> unconnected-(U13-PC1-Pad9)
Routing:
- net PWM4: track 22.6 -> 56.2 mm, vias 0 -> 2
- net MOTOR2b: track 137.6 -> 118.1 mm
- net MOTOR2a: track 137.5 -> 118.4 mm
- net PWM3: track 39.5 -> 50.8 mm
- net PWM2: track 36.8 -> 46.4 mm
- net MOTOR1a: track 105.9 -> 114.8 mm
- net PWM1: track 34.9 -> 39.0 mm
- net unconnected-(U13-PC3-Pad11): track 0.00 -> 0.88 mm
- net GND: track 802.8 -> 803.6 mm, vias 12 -> 255
- added copper zone on B.Cu, net GND
- added copper zone on F.Cu, net GND
