File: KiCAD/STM32 RC OVLADAČ/STM32 RC OVLADAČ.kicad_sch (KiCad schematic)
At the start: 17 parts, among them J1 USB_C_Receptacle_USB2.0_16P, U1 STM32F030C8Tx, U2 TP4056-42-ESOP8, U3 STM32F030C8Tx, U4 LD1117V33, U5 NRF24L01_Breakout, U6 NRF24L01_Breakout

Commit message: .
Parts:
- added J2, J3: Conn_01x05_Socket, Connector_Wire:SolderWire-0.5sqmm_1x05_P4.6mm_D0.9mm_OD2.1mm, symbol Connector:Conn_01x05_Socket
- added J4: Conn_01x04_Pin, symbol Connector:Conn_01x04_Pin
- added JP1, JP2, JP3, JP4, JP5, JP6, JP7, JP8: SolderJumper_3_Open, symbol Jumper:SolderJumper_3_Open
Connections:
- net +3.3V: now also U5.2 (VCC), U6.2 (VCC); no longer U3.9 (VDDA)
- net GND: now also U5.1 (GND), U6.1 (GND), J2.5 (Pin_5), J3.5 (Pin_5); no longer U3.8 (VSSA)
- net at U1.13 (PA3): now also U5.3 (CE)
- net at U1.14 (PA4): now also JP1.2 (C)
- net at U1.15 (PA5): now also JP2.2 (C)
- net at U1.16 (PA6): now also JP3.2 (C)
- net at U1.17 (PA7): now also JP4.2 (C)
- net at U5.4 (~{CSN}): now also JP1.3 (B)
- net at U5.5 (SCK): now also JP2.3 (B)
- net at U5.6 (MOSI): now also JP4.3 (B)
- net at U5.7 (MISO): now also JP3.3 (B)
- net at U3.13 (PA3): now also U6.3 (CE)
- net at U3.14 (PA4): now also JP5.2 (C)
- net at U3.15 (PA5): now also JP6.2 (C)
- net at U3.16 (PA6): now also JP7.2 (C)
- net at U3.17 (PA7): now also JP8.2 (C)
- net at U6.4 (~{CSN}): now also JP5.3 (B)
- net at U6.5 (SCK): now also JP6.3 (B)
- net at U6.6 (MOSI): now also JP8.3 (B)
- net at U6.7 (MISO): now also JP7.3 (B)
- new net: J3.1 (Pin_1), JP1.1 (A)
- new net: J3.2 (Pin_2), JP2.1 (A)
- new net: J3.3 (Pin_3), JP3.1 (A)
- new net: J3.4 (Pin_4), JP4.1 (A)
- new net: J2.2 (Pin_2), JP6.1 (A)
- new net: J2.3 (Pin_3), JP7.1 (A)
- new net: J2.4 (Pin_4), JP8.1 (A)
- new net: J2.1 (Pin_1), JP5.1 (A)
Other:
- moved on the sheet: BT1, C1, C2, D1, D2, R1, R2, R5, U1, U2, U3, U4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
